File: PCB-HOT-PLATE.kicad_sch (KiCad schematic)
At the start: 4 parts

Commit message: add Components
Parts:
- added C? (x2): 10u, symbol Device:C
- added C?: 0.1u, symbol Device:C
- added C?: 1u, symbol Device:C
- added J?: Conn_01x08, symbol Connector_Generic:Conn_01x08
- added J? (x2): Screw_Terminal_01x02, symbol Connector:Screw_Terminal_01x02
- added Q? (x2): S9013, symbol Device:Q_NPN_EBC
- added R?: 10k, symbol Device:R
- added RV?: R_Potentiometer, symbol Device:R_Potentiometer
- added S?: ADTSM65NVTR, ADTSM65NVTR, symbol ADTSM65NVTR:ADTSM65NVTR
- added U?: AMS1117-3.3, Package_TO_SOT_SMD:SOT-223-3_TabPin2, symbol Regulator_Linear:AMS1117-3.3
- added U?: CP2104, Package_DFN_QFN:QFN-24-1EP_4x4mm_P0.5mm_EP2.6x2.6mm, symbol Interface_USB:CP2104
- added U?: MAX6675, SOIC8, symbol SparkFun-AnalogIC:MAX6675
Connections:
- net D+: now also U?.3 (D+)
- net D-: now also U?.4 (D-)
- net EN: now also C?.1, Q?.3 (C), R?.2
- net GND: now also U?.49 (GND), C?.2, C?.2, J?.1 (Pin_1), J?.2 (Pin_2), RV?.3, U?.1 (GND), U?.1 (GND)
- net at U?.1 (VDDA), U?.43 (VDDA), U?.46 (VDDA): now also U?.2 (LNA_IN), U?.3 (VDDA3P3), U?.4 (VDDA3P3), C?.2, C?.2, R?.1
- net DC: now reaches U?.12 (IO32)
- net DC: now also J?.6 (Pin_6)
- net CS: now reaches U?.13 (IO33)
- net CS: now also J?.7 (Pin_7)
- net SDA: now reaches U?.15 (IO26)
- net SDA: now also J?.4 (Pin_4)
- net SCL: now reaches U?.18 (IO12)
- net SCL: now also J?.3 (Pin_3)
- net RES: now reaches U?.22 (IO2)
- net RES: now also J?.5 (Pin_5)
- net GPIO0: now reaches U?.23 (IO0)
- net GPIO0: now also Q?.3 (C)
- net Button: now reaches U?.25 (IO16)
- net Button: now also S?.4 (NO_2)
- net POTI: now reaches U?.35 (IO18)
- net POTI: now also RV?.2
- net TH_CS: now reaches U?.36 (IO23)
- net TH_CS: now also U?.6 (!CS)
- net TH_MIS0: now reaches U?.39 (IO22)
- net TH_MIS0: now also U?.7 ((MI)SO)
- net RX: now reaches U?.40 (U0RXD/IO3)
- net RX: now also U?.20 (RXD)
- net TX: now reaches U?.41 (U0TXD/IO1)
- net TX: now also U?.21 (TXD)
- net TH_SCK: now reaches U?.42 (IO21)
- net TH_SCK: now also U?.5 (SCK)
- net +5V renamed +3V3
- net +3V3: now also C?.1, C?.1, C?.1, J?.1 (Pin_1), J?.2 (Pin_2), J?.8 (Pin_8), RV?.1, S?.1 (COM_1), U?.2 (VO), U?.3 (VI), U?.4 (VCC), U?.7 (REGIN), U?.8 (VBUS), U?.9 (~{RST})
- new net: U?.2 (GND), U?.25 (GND)
- new net: U?.5 (VIO), U?.6 (VDD)
- new net: J?.2 (Pin_2), U?.2 (T-)
- new net: J?.1 (Pin_1), U?.3 (T+)
- new net DTR: Q?.1 (E), Q?.2 (B), U?.23 (~{DTR})
- new net RTS: Q?.1 (E), Q?.2 (B), U?.19 (~{RTS})
Other:
- note added: "3V3 Regulator"
- note added: "AUTORESET"
- note added: "Button"
- note added: "ESP32 PICO D4"
- note added: "PCB Hot Plate"
- note added: "Potentiometer"
- note added: "Power"
- note added: "TFT DISPLAY"
- note added: "Temperature Sensor"
- note added: "USB2SERIAL"
- moved on the sheet: P?, R?, U?
